Commit message: first integration with nav stack. new cobo_full* files

File: diffdrive_arduino-humble/description/urdf/diffbot_description.urdf_v5.xacro (robot description, xacro)
@@ -47,5 +47,5 @@
   </joint>
   <!-- Base Link -->
-  <link name="${prefix}base_link">
+  <link name="base_link">
     <collision>
       <origin xyz="0 0 1" rpy="0 0 0"/>
@@ -70,7 +70,7 @@
       </inertial>
     </link>
-    <joint name="${prefix}right_wheel_joint" type="continuous">
-      <parent link="${prefix}base_link"/>
-      <child link="${prefix}right_wheel"/>
+    <joint name="right_wheel_joint" type="continuous">
+      <parent link="base_link"/>
+      <child link="right_wheel"/>
       <origin xyz="-0.2 -${base_width/2-wheel_len} 0" rpy="0 0 0"/>
       <axis xyz="0 1 0"/>
@@ -78,5 +78,5 @@
     </joint>
     <!-- right wheel Link -->
-    <link name="${prefix}right_wheel">
+    <link name="right_wheel">
       <collision>
         <origin xyz="0 0 0" rpy="${PI/2} 0 0"/>
@@ -101,7 +101,7 @@
         </inertial>
       </link>
-    <joint name="${prefix}left_wheel_joint" type="continuous">
-      <parent link="${prefix}base_link"/>
-      <child link="${prefix}left_wheel"/>
+    <joint name="left_wheel_joint" type="continuous">
+      <parent link="base_link"/>
+      <child link="left_wheel"/>
       <origin xyz="-0.2 ${base_width/2-wheel_len} 0" rpy="0 0 0"/>
       <axis xyz="0 1 0"/>
@@ -109,5 +109,5 @@
     </joint>
     <!-- left wheel Link -->
-    <link name="${prefix}left_wheel">
+    <link name="left_wheel">
       <collision>
         <origin xyz="0 0 0" rpy="${PI/2} 0 0"/>
@@ -132,11 +132,11 @@
         </inertial>
     </link>
-    <joint name="${prefix}caster_wheel_joint" type="fixed">
-      <parent link="${prefix}base_link"/>
-      <child link="${prefix}caster_wheel"/>
+    <joint name="caster_wheel_joint" type="fixed">
+      <parent link="base_link"/>
+      <child link="caster_wheel"/>
       <origin xyz="${base_width/2 - caster_wheel_radius} 0 ${-caster_wheel_radius}" rpy="0 0 0"/>
     </joint>
     <!-- caster wheel Link -->
-    <link name="${prefix}caster_wheel">
+    <link name="caster_wheel">
       <collision>
         <origin xyz="0 0 0" rpy="0 0 0"/>
