Commit message: second full stack integration. Add some logging, make sure arms are safely positioned before calibrate, adding PICK validation code, add more trajectories

File: cobo_arm_control/description/ros2_control/cobo.ros2_control_macro.xacro (robot description, xacro)
@@ -33,12 +33,11 @@
         </state_interface>
         <state_interface name="position"/>
-         <state_interface name="velocity"/>
-     </joint>
+        <state_interface name="velocity"/>
+      </joint>
       <joint name="${prefix}A_J_S1_U_A_L1_TO_L2_B1">
         <command_interface name="position">
           <param name="min">${-pi/2}</param>
           <param name="max">${pi/2}</param>
-         <state_interface name="velocity"/>
-       </command_interface>
+        </command_interface>
         <state_interface name="position">
           <param name="initial_value">0.0</param>

File: cobo_arm_control/description/urdf/cobo_full.urdf.xacro (robot description, xacro)
@@ -8,4 +8,18 @@
   <!-- ros2_control: diff drive hardware -->
   <xacro:include filename="$(find diffdrive_arduino)/urdf/diffbot.ros2_control_v5.xacro" />
+  <!-- Arm macro (cobo_arm) and arm link properties -->
+  <xacro:include filename="cobo_arm.macro.xacro" />
+  <!-- Left arm -->
+  <xacro:cobo_arm prefix="left_" parent="base_link">
+    <origin xyz="${base_length/2} ${base_width/2} ${-base_height/2 - wheel_radius}" rpy="0 0 ${-PI/2}"/>
+  </xacro:cobo_arm>
+  <!-- Right arm -->
+  <xacro:cobo_arm prefix="right_" parent="base_link">
+    <origin xyz="${base_length/2} ${-base_width/2} ${-base_height/2 - wheel_radius}" rpy="0 0 ${-PI/2}"/>
+  </xacro:cobo_arm>
+  <!-- ros2_control: arm + GPIO hardware -->
+  <xacro:include filename="../ros2_control/cobo.ros2_control_macro.xacro" />
+  <!-- ros2_control: arm + GPIO (cobo_arm_control/RobotSystem hardware plugin) -->
+  <xacro:cobo_ros2_control name="arm" prefix="cobo_"/>
   <!-- ros2_control: diff drive (diffdrive_arduino/DiffDriveArduinoHardware plugin).
        prefix="" so it references left_wheel_joint / right_wheel_joint defined above. -->
